File: life_tracker.sch (KiCad schematic (older format))
At the start: 2 parts, among them J1 TACTILE-NAV-SWITCH

Commit message: Initial pass at schematic.
Parts:
- removed LED1: 7-SEGMENT-4DIGIT-GREEN-CC, 7-SEGMENT-4DIGIT-YOUNGSUN, symbol SparkFun-LED:7-SEGMENT-4DIGIT-10MM-KGREEN
- added C1: 0.1uF, Capacitor_SMD:C_0805_2012Metric_Pad1.18x1.45mm_HandSolder, symbol Device:C
- added R1, R2, R3: 4.7k, Resistor_SMD:R_1206_3216Metric_Pad1.30x1.75mm_HandSolder, symbol Device:R
- added R4, R5: 39k, Resistor_SMD:R_1206_3216Metric_Pad1.30x1.75mm_HandSolder, symbol Device:R
- added U1: WeMos_D1_mini, Module:WEMOS_D1_mini_light, symbol MCU_Module:WeMos_D1_mini
- added U10, U11, U12: 5611AH, Display_7Segment:7SegmentLED_LTS6760_LTS6780, symbol Display_Character:SM420561N
- added U13: LSHD-7803, Display_7Segment:HDSP-A151, symbol Display_Character:HDSP-7503
- added U2, U3: PTS526-tactile-button, MyFootprints:pts526-tactile-button, symbol MySymbols:PTS526-tactile-button
- added U4: MAX6959BAEE+, MyFootprints:MAX6959BAEE&plus_, symbol 2021-10-18_05-36-44:MAX6959BAEE+
- added U5, U6, U7, U8: BAW56, SOT95P240X110-3N, symbol BAW56:BAW56
- added U9: I2C_128x64_OLED, MyFootprints:I2C_128x64_OLED, symbol MySymbols:I2C_128x64_OLED
Connections:
- net labels added: +5V, GND
- wire segments 0 -> 141
Other:
- moved on the sheet: J1

Commit message: Finished second revision.
Parts:
- removed R5: 39k, Resistor_SMD:R_1206_3216Metric_Pad1.30x1.75mm_HandSolder, symbol Device:R
- removed U10, U11, U12: 5611AH, Display_7Segment:7SegmentLED_LTS6760_LTS6780, symbol Display_Character:SM420561N
- removed U13: LSHD-7803, Display_7Segment:HDSP-A151, symbol Display_Character:HDSP-7503
- removed U4: MAX6959BAEE+, MyFootprints:MAX6959BAEE&plus_, symbol 2021-10-18_05-36-44:MAX6959BAEE+
- removed U5, U6, U7, U8: BAW56, SOT95P240X110-3N, symbol BAW56:BAW56
- added C1: 10uF, Capacitor_SMD:C_0805_2012Metric_Pad1.18x1.45mm_HandSolder, symbol Device:C
- added LED1: 7-SEGMENT-4DIGIT-10MM-KGREEN-CC, 7-SEGMENT-4DIGIT-YOUNGSUN, symbol MySymbols:7-SEGMENT-4DIGIT-10MM-KGREEN-CC
- added RV1: 100k, MyFootprints:TC33-SMD-Trimpot, symbol Device:R_POT_Small
- added U3: AS1115-BSST, Package_SO:QSOP-24_3.9x8.7mm_P0.635mm, symbol Interface_Expansion:AS1115-BSST
- R4: value 39k -> 4.7k
- renumbered C1 to C2, U9 to U2, U2 to U4, U3 to U5
Connections:
- wire segments 141 -> 87
Other:
- moved on the sheet: J1
